File: v2/khada.kicad_sch (KiCad schematic)
At the start: 54 parts, among them J1 MJ-4PP-9, SW1 SW_Push, SW10 SW_Push, SW11 SW_Push, SW12 SW_Push, SW13 SW_Push, SW14 SW_Push, SW15 SW_Push, SW16 SW_Push, SW17 SW_Push, SW18 SW_Push, SW19 SW_Push, SW2 SW_Push, SW20 SW_Push, SW21 SW_Push, SW22 SW_Push, SW23 RotaryEncoder_Switch, SW3 SW_Push, SW4 SW_Push, SW5 SW_Push, SW6 SW_Push, SW7 SW_Push, SW8 SW_Push, SW9 SW_Push, U1 YAAJ_WeAct_BlackPill_Part_Lik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

Commit message: save before moving mcu out
Parts:
- added U (x2): (no value), symbol keebio:Hole
- U: renamed from SW7; value SW_Push -> (none); footprint marbastlib-mx:SW_MX_Reversible_1u_PadsOnBothLayers -> (none)
- U: renamed from SW11; value SW_Push -> (none); footprint marbastlib-mx:SW_MX_Reversible_1u_PadsOnBothLayers -> (none)
- U: renamed from SW15; value SW_Push -> (none); footprint marbastlib-mx:SW_MX_Reversible_1u_PadsOnBothLayers -> (none)
- U: renamed from SW19; value SW_Push -> (none); footprint marbastlib-mx:SW_MX_Reversible_1u_PadsOnBothLayers -> (none)
- U: renamed from SW1; value SW_Push -> (none); footprint marbastlib-mx:SW_MX_Reversible_1u_PadsOnBothLayers -> (none)
- U: renamed from D1; value D_Small -> (none); footprint acheron_Components:D_THT_7.62mm_copy -> (none)
- U: renamed from SW4; value SW_Push -> (none); footprint marbastlib-mx:SW_MX_Reversible_1u_PadsOnBothLayers -> (none)
- U: renamed from D4; value D_Small -> (none); footprint acheron_Components:D_THT_7.62mm_copy -> (none)
- U: renamed from SW8; value SW_Push -> (none); footprint marbastlib-mx:SW_MX_Reversible_1u_PadsOnBothLayers -> (none)
- U: renamed from D8; value D_Small -> (none); footprint acheron_Components:D_THT_7.62mm_copy -> (none)
- U: renamed from SW12; value SW_Push -> (none); footprint marbastlib-mx:SW_MX_Reversible_1u_PadsOnBothLayers -> (none)
- U: renamed from D12; value D_Small -> (none); footprint acheron_Components:D_THT_7.62mm_copy -> (none)
- U: renamed from SW16; value SW_Push -> (none); footprint marbastlib-mx:SW_MX_Reversible_1u_PadsOnBothLayers -> (none)
- U: renamed from D16; value D_Small -> (none); footprint acheron_Components:D_THT_7.62mm_copy -> (none)
- U: renamed from SW2; value SW_Push -> (none); footprint marbastlib-mx:SW_MX_Reversible_1u_PadsOnBothLayers -> (none)
- U: renamed from D2; value D_Small -> (none); footprint acheron_Components:D_THT_7.62mm_copy -> (none)
- U: renamed from SW5; value SW_Push -> (none); footprint marbastlib-mx:SW_MX_Reversible_1u_PadsOnBothLayers -> (none)
- U: renamed from D5; value D_Small -> (none); footprint acheron_Components:D_THT_7.62mm_copy -> (none)
- U: renamed from SW9; value SW_Push -> (none); footprint marbastlib-mx:SW_MX_Reversible_1u_PadsOnBothLayers -> (none)
- U: renamed from D9; value D_Small -> (none); footprint acheron_Components:D_THT_7.62mm_copy -> (none)
- U: renamed from SW13; value SW_Push -> (none); footprint marbastlib-mx:SW_MX_Reversible_1u_PadsOnBothLayers -> (none)
- U: renamed from D13; value D_Small -> (none); footprint acheron_Components:D_THT_7.62mm_copy -> (none)
- U: renamed from SW17; value SW_Push -> (none); footprint marbastlib-mx:SW_MX_Reversible_1u_PadsOnBothLayers -> (none)
- U: renamed from D17; value D_Small -> (none); footprint acheron_Components:D_THT_7.62mm_copy -> (none)
- U: renamed from SW21; value SW_Push -> (none); footprint marbastlib-mx:SW_MX_Reversible_1u_PadsOnBothLayers -> (none)
- U: renamed from D21; value D_Small -> (none); footprint acheron_Components:D_THT_7.62mm_copy -> (none)
- U: renamed from SW3; value SW_Push -> (none); footprint marbastlib-mx:SW_MX_Reversible_1u_PadsOnBothLayers -> (none)
- U: renamed from D3; value D_Small -> (none); footprint acheron_Components:D_THT_7.62mm_copy -> (none)
- U: renamed from SW6; value SW_Push -> (none); footprint marbastlib-mx:SW_MX_Reversible_1u_PadsOnBothLayers -> (none)
- U: renamed from D6; value D_Small -> (none); footprint acheron_Components:D_THT_7.62mm_copy -> (none)
- U: renamed from SW10; value SW_Push -> (none); footprint marbastlib-mx:SW_MX_Reversible_1u_PadsOnBothLayers -> (none)
- U: renamed from D10; value D_Small -> (none); footprint acheron_Components:D_THT_7.62mm_copy -> (none)
- U: renamed from SW14; value SW_Push -> (none); footprint marbastlib-mx:SW_MX_Reversible_1u_PadsOnBothLayers -> (none)
- U: renamed from D14; value D_Small -> (none); footprint acheron_Components:D_THT_7.62mm_copy -> (none)
- U: renamed from SW18; value SW_Push -> (none); footprint marbastlib-mx:SW_MX_Reversible_1u_PadsOnBothLayers -> (none)
- U: renamed from D18; value D_Small -> (none); footprint acheron_Components:D_THT_7.62mm_copy -> (none)
- U: renamed from SW22; value SW_Push -> (none); footprint marbastlib-mx:SW_MX_Reversible_1u_PadsOnBothLayers -> (none)
- U: renamed from D22; value D_Small -> (none); footprint acheron_Components:D_THT_7.62mm_copy -> (none)
- U: renamed from D7; value D_Small -> (none); footprint acheron_Components:D_THT_7.62mm_copy -> (none)
- U: renamed from D11; value D_Small -> (none); footprint acheron_Components:D_THT_7.62mm_copy -> (none)
- U: renamed from D15; value D_Small -> (none); footprint acheron_Components:D_THT_7.62mm_copy -> (none)
- U: renamed from D19; value D_Small -> (none); footprint acheron_Components:D_THT_7.62mm_copy -> (none)
- U: renamed from SW23; value RotaryEncoder_Switch -> (none); footprint keebio:RotaryEncoder_Alps_EC11E-Switch_Vertical_H20mm -> (none)
- U: renamed from H5; value Hole -> (none); footprint used_footprints:M2_HOLE_PCB -> (none)
- U: renamed from H1; value Hole -> (none); footprint used_footprints:M2_HOLE_PCB -> (none)
- U: renamed from H2; value Hole -> (none); footprint used_footprints:M2_HOLE_PCB -> (none)
- U: renamed from H3; value Hole -> (none); footprint used_footprints:M2_HOLE_PCB -> (none)
- U: renamed from U1; value YAAJ_WeAct_BlackPill_Part_Like_SWD_Breakout -> (none); footprint blackpills:YAAJ_WeAct_BlackPill_SWD_2 -> (none)
- U: renamed from D20; value D_Small -> (none); footprint acheron_Components:D_THT_7.62mm_copy -> (none)
- U: renamed from SW20; value SW_Push -> (none); footprint marbastlib-mx:SW_MX_Reversible_1u_PadsOnBothLayers -> (none)
- U: renamed from J1; value MJ-4PP-9 -> (none); footprint kbd:MJ-4PP-9 -> (none)
- U: renamed from R1; value 10k -> (none); footprint Resistor_THT:R_Axial_DIN0204_L3.6mm_D1.6mm_P5.08mm_Horizontal -> (none)
- U: renamed from D23; value D_Small -> (none); footprint acheron_Components:D_THT_7.62mm_copy -> (none)
- U: renamed from H4; value Hole -> (none); footprint used_footprints:M2_HOLE_PCB -> (none)
Connections:
- net +5V: now also U.2, U.40 (5V), U.D; no longer U.1, U.18 (5V), U.C
- net DATA: now also U.1, U.A; no longer U.2, U.B
- net GND: now also U.C; no longer U.D
Other:
- moved on the sheet: U

Commit message: add new switch for macros
Parts:
- removed U (x3): (no value), symbol keebio:Hole
- added U: (no value), symbol Device:D_Small
- added U: (no value), symbol Switch:SW_Push
Connections:
- net col0: now also U.2
- net col1: now also U.2; no longer U.2
- net col2: now also U.2; no longer U.2
- net col3: now also U.2; no longer U.2
- net col4: now also U.S2, U.1 (K); no longer U.2
- net col5: now also U.2; no longer U.S2
- new net: U.1, U.2 (A)
Other:
- moved on the sheet: U

Commit message: new sw placement, new macro sw, trrs jack now on top
Parts:
- added U (x2): (no value), symbol keebio:Hole
- U: symbol YAAJ_WeAct_BlackPill_Part_Like_SWD_Breakout:YAAJ_WeAct_BlackPill_Part_Like_SWD_Breakout -> YAAJ_WeAct_BlackPill_Part_Like:YAAJ_WeAct_BlackPill_Part_Like
Connections:
- net GND: no longer U.41 (GND)
- net ROTA: now also U.17 (PB9); no longer U.16 (PB8)
- net ROTB: now also U.16 (PB8); no longer U.17 (PB9)
- net col4: now also U.2; no longer U.1 (K), U.S2
- net col5: now also U.S2; no longer U.2
- net row3: now also U.1 (K)
Other:
- moved on the sheet: U
