File: v2/case/khada.kicad_pcb (KiCad board)
At the start: 2 copper layers, 157.5 x 115.4 mm, 23 parts, among them SW1 SW_Push, SW10 SW_Push, SW11 SW_Push, SW12 SW_Push, SW13 SW_Push, SW14 SW_Push, SW15 SW_Push, SW16 SW_Push, SW17 SW_Push, SW18 SW_Push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

Commit message: case updated
Parts:
- moved SW16 29.0 mm to (173.2, 130.1)
- moved SW23 29.0 mm to (142.3, 83.9)
- moved SW10 29.0 mm to (84.9, 63.4)
- moved SW14 29.0 mm to (104.1, 60.4)
- moved SW5 29.0 mm to (65.9, 54.5)
- moved SW1 29.0 mm to (46.8, 54.5)
- moved SW11 29.0 mm to (84.9, 82.5)
- moved SW13 29.0 mm to (104.1, 41.4)
- moved SW15 29.0 mm to (104.1, 79.5)
- moved SW4 29.0 mm to (106.0, 109.1)
- moved SW6 29.0 mm to (65.9, 73.6)
- moved SW7 29.0 mm to (65.9, 92.6)
- moved SW8 29.0 mm to (127.9, 109.8)
- moved SW9 29.0 mm to (84.9, 44.4)
- moved SW17 29.0 mm to (123.2, 44.6)
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Other:
- board size 157.5 x 115.4 mm -> 187.5 x 146.4 mm
